Commit message: before git ignore

File: src/arm_urdf/urdf/arm_urdf.xacro (robot description, xacro)
@@ -5,15 +5,33 @@
     <xacro:macro name="arm" params="prefix">
         <!-- links -->
+        <!-- <link name="${prefix}_base_fixed">
+            <visual>
+            <origin rpy="0 0 0" xyz="0 0 0.4"/>
+            <geometry>
+                <box size="0.3 0.5 1"/>
+            </geometry>
+            </visual>
+            <collision>
+            <origin rpy="0 0 0" xyz="0 0 0.4"/>
+            <geometry>
+                <box size="0.3 0.3 0.8"/>
+            </geometry>
+            </collision>
+            <inertial>
+            <mass value="0.5"/>
+            <inertia ixx="0.4" ixy="0.0" ixz="0.0" iyy="0.4" iyz="0.0" izz="0.2"/>
+            </inertial>
+        </link> -->
         <link name="${prefix}_base_fixed">
             <visual>
-            <origin rpy="0 0 0" xyz="0 0 0.4"/>
-            <geometry>
-                <box size="0.3 0.5 1"/>
-            </geometry>
-            </visual>
-            <collision>
-            <origin rpy="0 0 0" xyz="0 0 0.4"/>
-            <geometry>
-                <box size="0.3 0.3 0.8"/>
+            <origin rpy="0 0 0" xyz="0 0 0"/>
+            <geometry>
+                <box size="0.2 0.2 0.05"/>
+            </geometry>
+            </visual>
+            <collision>
+            <origin rpy="0 0 0" xyz="0 0 0"/>
+            <geometry>
+                <box size="0.18 0.18 0.03"/>
             </geometry>
             </collision>
@@ -154,6 +172,14 @@
         <!-- joints -->
         <!-- joint names defined like so: ${prefix}_<parent>_<child>_joint -->
+        <!-- <joint name="${prefix}_base_fixed_base_joint" type="revolute">
+            <origin rpy="0 ${radians(90)} 0" xyz="0.15 0 0.6"/>
+            <axis xyz="0 0 1"/>
+            <limit effort="1000.0" lower="${radians(-180)}" upper="${radians(180)}" velocity="2.5"/>
+            <parent link="${prefix}_base_fixed" />
+            <child link="${prefix}_base" />
+            <dynamics D="1" K="7000" mu_coulomb="0" mu_viscous="16" damping="0.003" friction="0.0"/>
+        </joint> -->
         <joint name="${prefix}_base_fixed_base_joint" type="revolute">
-            <origin rpy="0 ${radians(90)} 0" xyz="0.15 0 0.6"/>
+            <origin rpy="0 0 0" xyz="0 0 0.05"/>
             <axis xyz="0 0 1"/>
             <limit effort="1000.0" lower="${radians(-180)}" upper="${radians(180)}" velocity="2.5"/>

Commit message: changed original urdf model to have smaller base and vertically oriented arm, added kinect sensor to urdf and simulation, seperate test file for pick and place tests but tests still failing for picking up objects

File: src/arm_urdf/urdf/arm_urdf.xacro (robot description, xacro)
@@ -25,13 +25,13 @@
         <link name="${prefix}_base_fixed">
             <visual>
-            <origin rpy="0 0 0" xyz="0 0 0"/>
-            <geometry>
-                <box size="0.2 0.2 0.05"/>
-            </geometry>
-            </visual>
-            <collision>
-            <origin rpy="0 0 0" xyz="0 0 0"/>
-            <geometry>
-                <box size="0.18 0.18 0.03"/>
+            <origin rpy="0 0 0" xyz="0 0 0.025"/>
+            <geometry>
+                <box size="0.4 0.4 0.05"/>
+            </geometry>
+            </visual>
+            <collision>
+            <origin rpy="0 0 0" xyz="0 0 0.025"/>
+            <geometry>
+                <box size="0.4 0.4 0.05"/>
             </geometry>
             </collision>

File: src/arm_urdf/urdf/main.xacro (robot description, xacro)
@@ -26,3 +26,48 @@
         <child link="${arm_prefix}_base_fixed" />
     </joint>
+    <!--Kinect-->
+    <!-- position of kinect has to be changed in common_sensors/urdf/sensors/kinect_properties.urdf.xacro-->
+    <!-- <xacro:include filename="$(find common_sensors)/urdf/sensors/kinect.urdf.xacro" />
+    <xacro:sensor_kinect parent="world"/> -->
+    <gazebo reference="${arm_prefix}_camera_link">
+        <sensor name="${arm_prefix}_camera" type="depth">
+            <update_rate>20</update_rate>
+            <camera>
+            <horizontal_fov>1.047198</horizontal_fov>
+            <image>
+                <width>640</width>
+                <height>480</height>
+                <format>R8G8B8</format>
+            </image>
+            <clip>
+                <near>0.05</near>
+                <far>3</far>
+            </clip>
+            </camera>
+            <plugin name="${arm_prefix}_kinetic_camera_controller" filename="libgazebo_ros_openni_kinect.so">
+            <baseline>0.2</baseline>
+            <alwaysOn>true</alwaysOn>
+            <updateRate>1.0</updateRate>
+            <cameraName>${arm_prefix}_camera_ir</cameraName>
+            <imageTopicName>/${arm_prefix}_camera/color/image_raw</imageTopicName>
+            <cameraInfoTopicName>/${arm_prefix}_camera/color/camera_info</cameraInfoTopicName>
+            <depthImageTopicName>/${arm_prefix}_camera/depth/image_raw</depthImageTopicName>
+            <depthImageInfoTopicName>/${arm_prefix}_camera/depth/camera_info</depthImageInfoTopicName>
+            <pointCloudTopicName>/${arm_prefix}_camera/depth/points</pointCloudTopicName>
+            <frameName>${arm_prefix}_camera_link</frameName>
+            <pointCloudCutoff>0.5</pointCloudCutoff>
+            <pointCloudCutoffMax>3.0</pointCloudCutoffMax>
+            <distortionK1>0.00000001</distortionK1>
+            <distortionK2>0.00000001</distortionK2>
+            <distortionK3>0.00000001</distortionK3>
+            <distortionT1>0.00000001</distortionT1>
+            <distortionT2>0.00000001</distortionT2>
+            <CxPrime>0</CxPrime>
+            <Cx>0</Cx>
+            <Cy>0</Cy>
+            <focalLength>0</focalLength>
+            <hackBaseline>0</hackBaseline>
+            </plugin>
+        </sensor>
+    </gazebo>
 </robot>
