Commit message: arm with mobile base and simulation

File: ob1_arm_description/urdf/arm_with_base.xacro (robot description, xacro)
@@ -2,4 +2,5 @@
 <robot xmlns:xacro="http://www.ros.org/wiki/xacro" name="arm_with_pedestal">
     <xacro:property name="arm_name" value="arm1" />
+    <xacro:property name="base_name" value="base" />
     <xacro:property name="width" value="0.5" />
     <xacro:property name="height" value="1.7" />
@@ -14,10 +15,10 @@
             </geometry>
             </visual>
-            <collision>
-            <origin rpy="0 0 0" xyz="0 0 0.4"/>
+            <!-- <collision>
+            <origin rpy="0 0 0" xyz="0 0 ${height/2}"/>
             <geometry>
                 <box size="${width} ${width} ${height}"/>
             </geometry>
-            </collision>
+            </collision> -->
             <inertial>
                 <mass value="100" />
@@ -26,11 +27,16 @@
             </inertial>
         </link>
+        <joint name="hip_torso_joint" type="fixed">
+            <parent link="tele_hip_link"/>
+            <child link="torso"/>
+            <origin xyz="0 0 0.2" rpy="0 0 0"/>
+        </joint>
         <joint name="torso_base_joint" type="continuous">
             <origin rpy="${-pi/2} 0 0" xyz="0 ${width/2} ${height*2/3}"/>
             <axis xyz="0 0 1"/>
-            <!-- <limit effort="1000.0" lower="${radians(-180)}" upper="${radians(180)}" velocity="0.5"/> -->
+            <limit effort="1000.0" lower="${radians(-180)}" upper="${radians(180)}" velocity="0.5"/>
             <parent link="torso" />
             <child link="${arm_name}_base_link" />
-            <!-- <dynamics D="1" K="7000" mu_coulomb="0" mu_viscous="16" damping="0.003" friction="0.0"/> -->
+            <dynamics D="1" K="7000" mu_coulomb="0" mu_viscous="16" damping="0.003" friction="0.0"/>
         </joint>
         <link name="tele_hip_link">
@@ -59,9 +65,4 @@
             <origin xyz="0 0 0" rpy="0 0 0"/>
             <limit lower="0" upper="0.15" velocity="0.1" effort="1.0" />
-        </joint>
-        <joint name="hip_torso_joint" type="fixed">
-            <parent link="tele_hip_link"/>
-            <child link="torso"/>
-            <origin xyz="0 0 0.2" rpy="0 0 0"/>
         </joint>
         <link name="camera_link">
@@ -130,4 +131,5 @@
             </gazebo>
     </xacro:macro>
+    <xacro:mobile_base base_name="${base_name}"/>
     <xacro:arm arm_name="${arm_name}"/>
     <xacro:pedestal/>

File: ob1_arm_description/urdf/ob1_arm.xacro (robot description, xacro)
@@ -78,5 +78,5 @@
             <inertial>
                 <origin xyz="0 0 0" rpy="0 0 0"/>
-                <mass value="0" />
+                <mass value="1" />
                 <inertia ixx="0" ixy="0"  ixz="0" iyy="0" iyz="0" izz="0" />
             </inertial>
@@ -193,5 +193,5 @@
             <inertial>
                 <origin xyz="0 0 0" rpy="0 0 0"/>
-                <mass value="0" />
+                <mass value="1" />
                 <inertia ixx="0" ixy="0"  ixz="0" iyy="0" iyz="0" izz="0" />
             </inertial>
@@ -290,5 +290,5 @@
             <inertial>
                 <origin xyz="0 0 0" rpy="0 0 0"/>
-                <mass value="0" />
+                <mass value="1" />
                 <inertia ixx="0" ixy="0"  ixz="0" iyy="0" iyz="0" izz="0" />
             </inertial>
@@ -351,5 +351,5 @@
             <inertial>
                 <origin xyz="0 0 0" rpy="0 0 0"/>
-                <mass value="0" />
+                <mass value="1" />
                 <inertia ixx="0" ixy="0"  ixz="0" iyy="0" iyz="0" izz="0" />
             </inertial>
@@ -430,5 +430,5 @@
             <inertial>
                 <origin xyz="0 0 0" rpy="0 0 0"/>
-                <mass value="0" />
+                <mass value="1" />
                 <inertia ixx="0" ixy="0"  ixz="0" iyy="0" iyz="0" izz="0" />
             </inertial>
@@ -1373,5 +1373,5 @@
             <inertial>
                 <origin xyz="0 0 0" rpy="0 0 0"/>
-                <mass value="0" />
+                <mass value="1" />
                 <inertia ixx="0" ixy="0"  ixz="0" iyy="0" iyz="0" izz="0" />
             </inertial>

Commit message: physics and gazebo changes to arm description

File: ob1_arm_description/urdf/arm_with_base.xacro (robot description, xacro)
@@ -7,4 +7,5 @@
     <xacro:include filename="$(find ob1_arm_description)/urdf/ob1_arm.xacro"/>
     <xacro:include filename="$(find ob1_arm_description)/urdf/mobile_base.xacro"/>
+    <xacro:include filename="$(find ob1_arm_description)/urdf/ob1_arm_gazebo.xacro"/>
     <xacro:macro name="pedestal">
         <link name="torso">
@@ -68,5 +69,5 @@
         <link name="camera_link">
             <visual>
-            <origin rpy="${pi/4} 0 0" xyz="0 0 0"/>
+            <origin rpy="${-pi/2} 0 0" xyz="0 0 0"/>
             <geometry>
                 <box size="0.1 0.1 0.1"/>

File: ob1_arm_description/urdf/arm_with_pedestal.xacro (robot description, xacro)
@@ -129,6 +129,10 @@
             </sensor>
             </gazebo>
+        <gazebo reference="torso">
+            <selfCollide>true</selfCollide>
+        </gazebo>
     </xacro:macro>
     <xacro:arm arm_name="${arm_name}"/>
+    <xacro:arm_gazebo arm_name="${arm_name}"/>
     <xacro:pedestal/>
 </robot>

File: ob1_arm_description/urdf/ob1_arm.xacro (robot description, xacro)
@@ -79,5 +79,5 @@
                 <origin xyz="0 0 0" rpy="0 0 0"/>
                 <mass value="1" />
-                <inertia ixx="0" ixy="0"  ixz="0" iyy="0" iyz="0" izz="0" />
+                <inertia ixx="0.4" ixy="0.0" ixz="0.0" iyy="0.4" iyz="0.0" izz="0.2"/>
             </inertial>
         </link>
@@ -194,5 +194,5 @@
                 <origin xyz="0 0 0" rpy="0 0 0"/>
                 <mass value="1" />
-                <inertia ixx="0" ixy="0"  ixz="0" iyy="0" iyz="0" izz="0" />
+                <inertia ixx="0.4" ixy="0.0" ixz="0.0" iyy="0.4" iyz="0.0" izz="0.2"/>
             </inertial>
         </link>
@@ -291,5 +291,5 @@
                 <origin xyz="0 0 0" rpy="0 0 0"/>
                 <mass value="1" />
-                <inertia ixx="0" ixy="0"  ixz="0" iyy="0" iyz="0" izz="0" />
+                <inertia ixx="0.4" ixy="0.0" ixz="0.0" iyy="0.4" iyz="0.0" izz="0.2"/>
             </inertial>
         </link>
@@ -352,5 +352,5 @@
                 <origin xyz="0 0 0" rpy="0 0 0"/>
                 <mass value="1" />
-                <inertia ixx="0" ixy="0"  ixz="0" iyy="0" iyz="0" izz="0" />
+                <inertia ixx="0.4" ixy="0.0" ixz="0.0" iyy="0.4" iyz="0.0" izz="0.2"/>
             </inertial>
         </link>
@@ -431,5 +431,5 @@
                 <origin xyz="0 0 0" rpy="0 0 0"/>
                 <mass value="1" />
-                <inertia ixx="0" ixy="0"  ixz="0" iyy="0" iyz="0" izz="0" />
+                <inertia ixx="0.4" ixy="0.0" ixz="0.0" iyy="0.4" iyz="0.0" izz="0.2"/>
             </inertial>
         </link>
@@ -1374,5 +1374,5 @@
                 <origin xyz="0 0 0" rpy="0 0 0"/>
                 <mass value="1" />
-                <inertia ixx="0" ixy="0"  ixz="0" iyy="0" iyz="0" izz="0" />
+                <inertia ixx="0.4" ixy="0.0" ixz="0.0" iyy="0.4" iyz="0.0" izz="0.2"/>
             </inertial>
         </link>
