Commit message: new gripper

File: ob1_arm_description/urdf/ob1_arm_gazebo.xacro (robot description, xacro)
@@ -1,21 +1,21 @@
 <?xml version="1.0"?>
 <robot xmlns:xacro="http://www.ros.org/wiki/xacro" name="ob1_arm">
-    <xacro:macro name="arm_gazebo" params="arm_name">
-        <gazebo reference="${arm_name}_base_link">
+    <xacro:macro name="arm_gazebo" params="prefix">
+        <gazebo reference="${prefix}_base_link">
             <selfCollide>true</selfCollide>
         </gazebo>
-        <gazebo reference="shoulder_link">
+        <gazebo reference="${prefix}_shoulder_link">
             <selfCollide>true</selfCollide>
         </gazebo>
-        <gazebo reference="arm_link">
+        <gazebo reference="${prefix}_arm_link">
             <selfCollide>true</selfCollide>
         </gazebo>
-        <gazebo reference="elbow_link">
+        <gazebo reference="${prefix}_elbow_link">
             <selfCollide>true</selfCollide>
         </gazebo>
-        <gazebo reference="forearm_link">
+        <gazebo reference="${prefix}_forearm_link">
             <selfCollide>true</selfCollide>
         </gazebo>
-        <gazebo reference="main_assembly">
+        <gazebo reference="${prefix}_gripper_assembly_link">
             <selfCollide>true</selfCollide>
         </gazebo>

File: ob1_arm_description/urdf/old/ob1_arm.urdf (robot description, URDF)
Before this commit: robot ob1_arm, 6 links, 5 joints
Links:
- link arm_link: geometry collision mesh filename=package://ob1_arm_description/meshes/arm/bicep_linkage_-_en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; collision mesh filename=package://ob1_arm_description/meshes/arm/bicep_linkage_-_mo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
- link base_link: geometry collision mesh filename=package://ob1_arm_description/meshes/arm/motor_front_suppor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; collision mesh filename=package://ob1_arm_description/meshes/arm/motor_mid_support_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
- link elbow_link: geometry collision mesh filename=package://ob1_arm_description/meshes/arm/forearm_intermedia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; collision mesh filename=package://ob1_arm_description/meshes/arm/forearm_motor_supp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
- link forearm_link: geometry collision mesh filename=package://ob1_arm_description/meshes/arm/end_effector_plate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; collision mesh filename=package://ob1_arm_description/meshes/arm/forearm_linkage_-_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
- link main_assembly: geometry collision mesh filename=package://ob1_arm_description/meshes/arm/535198.stl; collision mesh filename=package://ob1_arm_description/meshes/arm/535198.stl
- link shoulder_link: geometry collision mesh filename=package://ob1_arm_description/meshes/arm/bicep_plate_-_real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; collision mesh filename=package://ob1_arm_description/meshes/arm/bicep_y_motor.stl
