Commit message: new gripper

File: ob1_arm_description/urdf/old/ob1_arm.xacro (robot description, xacro)
@@ -7,5 +7,5 @@
                 <origin xyz="3.31402e-16 -0.0195 0.06" rpy="-1.5708 1.21431e-16 3.90606e-18" />
                 <geometry>
-                    <mesh filename="package://ob1_arm_description/meshes/shoulder_y_motor.stl"/>
+                    <mesh filename="package://ob1_arm_description/meshes/arm/shoulder_y_motor.stl"/>
                 </geometry>
                 <material name="shoulder_y_motor_material">
@@ -16,5 +16,5 @@
                 <origin xyz="3.31402e-16 -0.0195 0.06" rpy="-1.5708 1.21431e-16 3.90606e-18" />
                 <geometry>
-                    <mesh filename="package://ob1_arm_description/meshes/shoulder_y_motor.stl"/>
+                    <mesh filename="package://ob1_arm_description/meshes/arm/shoulder_y_motor.stl"/>
                 </geometry>
                 <material name="shoulder_y_motor_material">
@@ -25,5 +25,5 @@
                 <origin xyz="1.33481e-16 -0.0195 0.06" rpy="-1.5708 1.2013e-16 2.92997e-21" />
                 <geometry>
-                    <mesh filename="package://ob1_arm_description/meshes/shoulder_plate.stl"/>
+                    <mesh filename="package://ob1_arm_description/meshes/arm/shoulder_plate.stl"/>
                 </geometry>
                 <material name="shoulder_plate_material">
@@ -34,5 +34,5 @@
                 <origin xyz="1.33481e-16 -0.0195 0.06" rpy="-1.5708 1.2013e-16 2.92997e-21" />
                 <geometry>
-                    <mesh filename="package://ob1_arm_description/meshes/shoulder_plate.stl"/>
+                    <mesh filename="package://ob1_arm_description/meshes/arm/shoulder_plate.stl"/>
                 </geometry>
                 <material name="shoulder_plate_material">
@@ -43,5 +43,5 @@
                 <origin xyz="3.46418e-16 -0.0195 0.06" rpy="-1.5708 1.20997e-16 7.25353e-18" />
                 <geometry>
-                    <mesh filename="package://ob1_arm_description/meshes/motor_front_support_-_shoulder.stl"/>
+                    <mesh filename="package://ob1_arm_description/meshes/arm/motor_front_support_-_shoulder.stl"/>
                 </geometry>
                 <material name="motor_front_support_-_shoulder_material">
@@ -52,5 +52,5 @@
                 <origin xyz="3.46418e-16 -0.0195 0.06" rpy="-1.5708 1.20997e-16 7.25353e-18" />
                 <geometry>
-                    <mesh filename="package://ob1_arm_description/meshes/motor_front_support_-_shoulder.stl"/>
+                    <mesh filename="package://ob1_arm_description/meshes/arm/motor_front_support_-_shoulder.stl"/>
                 </geometry>
                 <material name="motor_front_support_-_shoulder_material">
@@ -61,5 +61,5 @@
                 <origin xyz="-6.0185e-17 -0.0195 0.06" rpy="-1.5708 1.20997e-16 7.25353e-18" />
                 <geometry>
-                    <mesh filename="package://ob1_arm_description/meshes/motor_mid_support_-_shoulder.stl"/>
+                    <mesh filename="package://ob1_arm_description/meshes/arm/motor_mid_support_-_shoulder.stl"/>
                 </geometry>
                 <material name="motor_mid_support_-_shoulder_material">
@@ -70,5 +70,5 @@
                 <origin xyz="-6.0185e-17 -0.0195 0.06" rpy="-1.5708 1.20997e-16 7.25353e-18" />
                 <geometry>
-                    <mesh filename="package://ob1_arm_description/meshes/motor_mid_support_-_shoulder.stl"/>
+                    <mesh filename="package://ob1_arm_description/meshes/arm/motor_mid_support_-_shoulder.stl"/>
                 </geometry>
                 <material name="motor_mid_support_-_shoulder_material">
@@ -86,5 +86,5 @@
                 <origin xyz="0 0 0.067" rpy="3.14159 3.60029e-32 -1.5708" />
                 <geometry>
-                    <mesh filename="package://ob1_arm_description/meshes/shoulder_linkage_-_motor.stl"/>
+                    <mesh filename="package://ob1_arm_description/meshes/arm/shoulder_linkage_-_motor.stl"/>
                 </geometry>
                 <material name="shoulder_linkage_-_motor_material">
@@ -95,5 +95,5 @@
                 <origin xyz="0 0 0.067" rpy="3.14159 3.60029e-32 -1.5708" />
                 <geometry>
-                    <mesh filename="package://ob1_arm_description/meshes/shoulder_linkage_-_motor.stl"/>
+                    <mesh filename="package://ob1_arm_description/meshes/arm/shoulder_linkage_-_motor.stl"/>
                 </geometry>
                 <material name="shoulder_linkage_-_motor_material">
@@ -104,5 +104,5 @@
                 <origin xyz="-6.03684e-16 -1.84994e-15 0.067" rpy="3.14159 7.97526e-16 -1.5708" />
                 <geometry>
-                    <mesh filename="package://ob1_arm_description/meshes/bicep_y_motor.stl"/>
+                    <mesh filename="package://ob1_arm_description/meshes/arm/bicep_y_motor.stl"/>
                 </geometry>
                 <material name="bicep_y_motor_material">
@@ -113,5 +113,5 @@
                 <origin xyz="-6.03684e-16 -1.84994e-15 0.067" rpy="3.14159 7.97526e-16 -1.5708" />
                 <geometry>
-                    <mesh filename="package://ob1_arm_description/meshes/bicep_y_motor.stl"/>
+                    <mesh filename="package://ob1_arm_description/meshes/arm/bicep_y_motor.stl"/>
                 </geometry>
                 <material name="bicep_y_motor_material">
@@ -122,5 +122,5 @@
                 <origin xyz="-1.31839e-16 -1.36238e-15 0.067" rpy="3.14159 -2.30393e-18 -1.5708" />
                 <geometry>
-                    <mesh filename="package://ob1_arm_description/meshes/motor_mid_support_-_bicep.stl"/>
+                    <mesh filename="package://ob1_arm_description/meshes/arm/motor_mid_support_-_bicep.stl"/>
                 </geometry>
                 <material name="motor_mid_support_-_bicep_material">
@@ -131,5 +131,5 @@
                 <origin xyz="-1.31839e-16 -1.36238e-15 0.067" rpy="3.14159 -2.30393e-18 -1.5708" />
                 <geometry>
-                    <mesh filename="package://ob1_arm_description/meshes/motor_mid_support_-_bicep.stl"/>
+                    <mesh filename="package://ob1_arm_description/meshes/arm/motor_mid_support_-_bicep.stl"/>
                 </geometry>
                 <material name="motor_mid_support_-_bicep_material">
@@ -140,5 +140,5 @@
                 <origin xyz="-7.70217e-16 -1.56706e-15 0.067" rpy="-3.14159 2.79702e-30 -1.5708" />
                 <geometry>
-                    <mesh filename="package://ob1_arm_description/meshes/bicep_plate_-_real.stl"/>
+                    <mesh filename="package://ob1_arm_description/meshes/arm/bicep_plate_-_real.stl"/>
                 </geometry>
                 <material name="bicep_plate_-_real_material">
@@ -149,5 +149,5 @@
                 <origin xyz="-7.70217e-16 -1.56706e-15 0.067" rpy="-3.14159 2.79702e-30 -1.5708" />
                 <geometry>
-                    <mesh filename="package://ob1_arm_description/meshes/bicep_plate_-_real.stl"/>
+                    <mesh filename="package://ob1_arm_description/meshes/arm/bicep_plate_-_real.stl"/>
                 </geometry>
                 <material name="bicep_plate_-_real_material">
@@ -158,5 +158,5 @@
                 <origin xyz="-2.42861e-16 -2.01669e-15 0.067" rpy="3.14159 3.86179e-16 -1.5708" />
                 <geometry>
-                    <mesh filename="package://ob1_arm_description/meshes/shoulder_linkage_-_encoder.stl"/>
+                    <mesh filename="package://ob1_arm_description/meshes/arm/shoulder_linkage_-_encoder.stl"/>
                 </geometry>
                 <material name="shoulder_linkage_-_encoder_material">
@@ -167,5 +167,5 @@
                 <origin xyz="-2.42861e-16 -2.01669e-15 0.067" rpy="3.14159 3.86179e-16 -1.5708" />
                 <geometry>
-                    <mesh filename="package://ob1_arm_description/meshes/shoulder_linkage_-_encoder.stl"/>
+                    <mesh filename="package://ob1_arm_description/meshes/arm/shoulder_linkage_-_encoder.stl"/>
                 </geometry>
                 <material name="shoulder_linkage_-_encoder_material">
@@ -176,5 +176,5 @@
                 <origin xyz="-2.70617e-16 -1.98014e-15 0.067" rpy="3.14159 2.23806e-16 -1.5708" />
                 <geometry>
-                    <mesh filename="package://ob1_arm_description/meshes/motor_front_support_-_bicep.stl"/>
+                    <mesh filename="package://ob1_arm_description/meshes/arm/motor_front_support_-_bicep.stl"/>
                 </geometry>
                 <material name="motor_front_support_-_bicep_material">
@@ -185,5 +185,5 @@
                 <origin xyz="-2.70617e-16 -1.98014e-15 0.067" rpy="3.14159 2.23806e-16 -1.5708" />
                 <geometry>
-                    <mesh filename="package://ob1_arm_description/meshes/motor_front_support_-_bicep.stl"/>
+                    <mesh filename="package://ob1_arm_description/meshes/arm/motor_front_support_-_bicep.stl"/>
                 </geometry>
                 <material name="motor_front_support_-_bicep_material">
@@ -201,5 +201,5 @@
                 <origin xyz="0.000575841 -1.05471e-15 0.0669915" rpy="3.14159 0.0295346 -7.29078e-16" />
                 <geometry>
-                    <mesh filename="package://ob1_arm_description/meshes/forearm_z_motor_shaft_collar_-_9604t12_flange-mount_shaft_collar.stl"/>
+                    <mesh filename="package://ob1_arm_description/meshes/arm/forearm_z_motor_shaft_collar_-_9604t12_flange-mount_shaft_collar.stl"/>
                 </geometry>
                 <material name="forearm_z_motor_shaft_collar_-_9604t12_flange-mount_shaft_collar_material">
@@ -210,5 +210,5 @@
                 <origin xyz="0.000575841 -1.05471e-15 0.0669915" rpy="3.14159 0.0295346 -7.29078e-16" />
                 <geometry>
-                    <mesh filename="package://ob1_arm_description/meshes/forearm_z_motor_shaft_collar_-_9604t12_flange-mount_shaft_collar.stl"/>
+                    <mesh filename="package://ob1_arm_description/meshes/arm/forearm_z_motor_shaft_collar_-_9604t12_flange-mount_shaft_collar.stl"/>
                 </geometry>
                 <material name="forearm_z_motor_shaft_collar_-_9604t12_flange-mount_shaft_collar_material">
@@ -219,5 +219,5 @@
                 <origin xyz="-9.25466e-16 1.55431e-15 0.067" rpy="3.14159 -4.40079e-18 -5.04871e-29" />
                 <geometry>
-                    <mesh filename="package://ob1_arm_description/meshes/bicep_z_motor.stl"/>
+                    <mesh filename="package://ob1_arm_description/meshes/arm/bicep_z_motor.stl"/>
                 </geometry>
                 <material name="bicep_z_motor_material">
@@ -228,5 +228,5 @@
                 <origin xyz="-9.25466e-16 1.55431e-15 0.067" rpy="3.14159 -4.40079e-18 -5.04871e-29" />
                 <geometry>
-                    <mesh filename="package://ob1_arm_description/meshes/bicep_z_motor.stl"/>
+                    <mesh filename="package://ob1_arm_description/meshes/arm/bicep_z_motor.stl"/>
                 </geometry>
                 <material name="bicep_z_motor_material">
@@ -237,5 +237,5 @@
                 <origin xyz="-9.99424e-16 -1.66533e-16 0.067" rpy="3.14159 -2.72597e-18 4.33681e-19" />
                 <geometry>
-                    <mesh filename="package://ob1_arm_description/meshes/bicep_linkage_-_encoder.stl"/>
+                    <mesh filename="package://ob1_arm_description/meshes/arm/bicep_linkage_-_encoder.stl"/>
                 </geometry>
                 <material name="bicep_linkage_-_encoder_material">
@@ -246,5 +246,5 @@
                 <origin xyz="-9.99424e-16 -1.66533e-16 0.067" rpy="3.14159 -2.72597e-18 4.33681e-19" />
                 <geometry>
-                    <mesh filename="package://ob1_arm_description/meshes/bicep_linkage_-_encoder.stl"/>
+                    <mesh filename="package://ob1_arm_description/meshes/arm/bicep_linkage_-_encoder.stl"/>
                 </geometry>
                 <material name="bicep_linkage_-_encoder_material">
@@ -255,5 +255,5 @@
                 <origin xyz="7.88861e-30 2.77556e-17 0.067" rpy="3.14159 4.93271e-31 0" />
                 <geometry>
-                    <mesh filename="package://ob1_arm_description/meshes/bicep_linkage_-_motor.stl"/>
+                    <mesh filename="package://ob1_arm_description/meshes/arm/bicep_linkage_-_motor.stl"/>
                 </geometry>
                 <material name="bicep_linkage_-_motor_material">
@@ -264,5 +264,5 @@
                 <origin xyz="7.88861e-30 2.77556e-17 0.067" rpy="3.14159 4.93271e-31 0" />
                 <geometry>
-                    <mesh filename="package://ob1_arm_description/meshes/bicep_linkage_-_motor.stl"/>
+                    <mesh filename="package://ob1_arm_description/meshes/arm/bicep_linkage_-_motor.stl"/>
                 </geometry>
                 <material name="bicep_linkage_-_motor_material">
@@ -273,5 +273,5 @@
                 <origin xyz="-8.25064e-16 1.05471e-15 0.067" rpy="3.14159 -3.17094e-18 -2.52435e-29" />
                 <geometry>
-                    <mesh filename="package://ob1_arm_description/meshes/forearm_plate.stl"/>
+                    <mesh filename="package://ob1_arm_description/meshes/arm/forearm_plate.stl"/>
                 </geometry>
                 <material name="forearm_plate_material">
@@ -282,5 +282,5 @@
                 <origin xyz="-8.25064e-16 1.05471e-15 0.067" rpy="3.14159 -3.17094e-18 -2.52435e-29" />
                 <geometry>
-                    <mesh filename="package://ob1_arm_description/meshes/forearm_plate.stl"/>
+                    <mesh filename="package://ob1_arm_description/meshes/arm/forearm_plate.stl"/>
                 </geometry>
                 <material name="forearm_plate_material">
@@ -298,5 +298,5 @@
                 <origin xyz="-4.05204e-16 0.0195 0.18" rpy="1.5708 2.52435e-29 -3.46945e-18" />
                 <geometry>
-                    <mesh filename="package://ob1_arm_description/meshes/forearm_motor_support.stl"/>
+                    <mesh filename="package://ob1_arm_description/meshes/arm/forearm_motor_support.stl"/>
                 </geometry>
                 <material name="forearm_motor_support_material">
@@ -307,5 +307,5 @@
                 <origin xyz="-4.05204e-16 0.0195 0.18" rpy="1.5708 2.52435e-29 -3.46945e-18" />
                 <geometry>
-                    <mesh filename="package://ob1_arm_description/meshes/forearm_motor_support.stl"/>
+                    <mesh filename="package://ob1_arm_description/meshes/arm/forearm_motor_support.stl"/>
                 </geometry>
                 <material name="forearm_motor_support_material">
@@ -316,5 +316,5 @@
                 <origin xyz="-1.25056e-17 0.0195 0.18" rpy="1.5708 2.52435e-29 3.23731e-28" />
                 <geometry>
-                    <mesh filename="package://ob1_arm_description/meshes/forearm_intermediate_plate.stl"/>
+                    <mesh filename="package://ob1_arm_description/meshes/arm/forearm_intermediate_plate.stl"/>
                 </geometry>
                 <material name="forearm_intermediate_plate_material">
@@ -325,5 +325,5 @@
                 <origin xyz="-1.25056e-17 0.0195 0.18" rpy="1.5708 2.52435e-29 3.23731e-28" />
                 <geometry>
-                    <mesh filename="package://ob1_arm_description/meshes/forearm_intermediate_plate.stl"/>
+                    <mesh filename="package://ob1_arm_description/meshes/arm/forearm_intermediate_plate.stl"/>
                 </geometry>
                 <material name="forearm_intermediate_plate_material">
@@ -334,5 +334,5 @@
                 <origin xyz="-6.05219e-16 0.05285 -0.03115" rpy="1.5708 2.52435e-29 -6.93889e-18" />
                 <geometry>
-                    <mesh filename="package://ob1_arm_description/meshes/part_1.stl"/>
+                    <mesh filename="package://ob1_arm_description/meshes/arm/part_1.stl"/>
                 </geometry>
                 <material name="part_1_material">
@@ -343,5 +343,5 @@
                 <origin xyz="-6.05219e-16 0.05285 -0.03115" rpy="1.5708 2.52435e-29 -6.93889e-18" />
                 <geometry>
-                    <mesh filename="package://ob1_arm_description/meshes/part_1.stl"/>
+                    <mesh filename="package://ob1_arm_description/meshes/arm/part_1.stl"/>
                 </geometry>
                 <material name="part_1_material">
@@ -359,5 +359,5 @@
                 <origin xyz="-5.02684e-16 0.21115 0.06335" rpy="7.88861e-31 -6.93889e-18 4.33681e-19" />
                 <geometry>
-                    <mesh filename="package://ob1_arm_description/meshes/end_effector_plate.stl"/>
+                    <mesh filename="package://ob1_arm_description/meshes/arm/end_effector_plate.stl"/>
                 </geometry>
                 <material name="end_effector_plate_material">
@@ -368,5 +368,5 @@
                 <origin xyz="-5.02684e-16 0.21115 0.06335" rpy="7.88861e-31 -6.93889e-18 4.33681e-19" />
                 <geometry>
-                    <mesh filename="package://ob1_arm_description/meshes/end_effector_plate.stl"/>
+                    <mesh filename="package://ob1_arm_description/meshes/arm/end_effector_plate.stl"/>
                 </geometry>
                 <material name="end_effector_plate_material">
@@ -377,5 +377,5 @@
                 <origin xyz="-2.79121e-16 0.21115 0.06335" rpy="3.15544e-30 1.08247e-15 3.90313e-18" />
                 <geometry>
-                    <mesh filename="package://ob1_arm_description/meshes/forearm_linkage_-_encoder.stl"/>
+                    <mesh filename="package://ob1_arm_description/meshes/arm/forearm_linkage_-_encoder.stl"/>
                 </geometry>
                 <material name="forearm_linkage_-_encoder_material">
@@ -386,5 +386,5 @@
                 <origin xyz="-2.79121e-16 0.21115 0.06335" rpy="3.15544e-30 1.08247e-15 3.90313e-18" />
                 <geometry>
-                    <mesh filename="package://ob1_arm_description/meshes/forearm_linkage_-_encoder.stl"/>
+                    <mesh filename="package://ob1_arm_description/meshes/arm/forearm_linkage_-_encoder.stl"/>
                 </geometry>
                 <material name="forearm_linkage_-_encoder_material">
@@ -395,5 +395,5 @@
                 <origin xyz="-1.00221e-17 0.21115 0.06335" rpy="7.88861e-31 -3.46945e-18 2.52435e-29" />
                 <geometry>
-                    <mesh filename="package://ob1_arm_description/meshes/forearm_linkage_-_motor.stl"/>
+                    <mesh filename="package://ob1_arm_description/meshes/arm/forearm_linkage_-_motor.stl"/>
                 </geometry>
                 <material name="forearm_linkage_-_motor_material">
@@ -404,5 +404,5 @@
                 <origin xyz="-1.00221e-17 0.21115 0.06335" rpy="7.88861e-31 -3.46945e-18 2.52435e-29" />
                 <geometry>
-                    <mesh filename="package://ob1_arm_description/meshes/forearm_linkage_-_motor.stl"/>
+                    <mesh filename="package://ob1_arm_description/meshes/arm/forearm_linkage_-_motor.stl"/>
                 </geometry>
                 <material name="forearm_linkage_-_motor_material">
@@ -413,5 +413,5 @@
                 <origin xyz="-5.17754e-16 0.21115 0.06335" rpy="1.57772e-30 1.07553e-15 3.90313e-18" />
                 <geometry>
-                    <mesh filename="package://ob1_arm_description/meshes/wrist_z_motor.stl"/>
+                    <mesh filename="package://ob1_arm_description/meshes/arm/wrist_z_motor.stl"/>
                 </geometry>
                 <material name="wrist_z_motor_material">
@@ -422,5 +422,5 @@
                 <origin xyz="-5.17754e-16 0.21115 0.06335" rpy="1.57772e-30 1.07553e-15 3.90313e-18" />
                 <geometry>
-                    <mesh filename="package://ob1_arm_description/meshes/wrist_z_motor.stl"/>
+                    <mesh filename="package://ob1_arm_description/meshes/arm/wrist_z_motor.stl"/>
                 </geometry>
                 <material name="wrist_z_motor_material">
@@ -438,5 +438,5 @@
                 <origin xyz="-0.0645733 -0.0670487 0.129369" rpy="-1.45249 0.81946 0.0866409" />
                 <geometry>
-                    <mesh filename="package://ob1_arm_description/meshes/part_1.stl"/>
+                    <mesh filename="package://ob1_arm_description/meshes/arm/part_1.stl"/>
                 </geometry>
                 <material name="part_1_material">
@@ -447,5 +447,5 @@
                 <origin xyz="-0.0645733 -0.0670487 0.129369" rpy="-1.45249 0.81946 0.0866409" />
                 <geometry>
-                    <mesh filename="package://ob1_arm_description/meshes/part_1.stl"/>
+                    <mesh filename="package://ob1_arm_description/meshes/arm/part_1.stl"/>
                 </geometry>
                 <material name="part_1_material">
@@ -456,5 +456,5 @@
                 <origin xyz="-0.0793646 0.0346641 0.226122" rpy="-1.60498 1.07372 -0.0300488" />
                 <geometry>
-                    <mesh filename="package://ob1_arm_description/meshes/part_1.stl"/>
+                    <mesh filename="package://ob1_arm_description/meshes/arm/part_1.stl"/>
                 </geometry>
                 <material name="part_1_material">
@@ -465,5 +465,5 @@
                 <origin xyz="-0.0793646 0.0346641 0.226122" rpy="-1.60498 1.07372 -0.0300488" />
                 <geometry>
-                    <mesh filename="package://ob1_arm_description/meshes/part_1.stl"/>
+                    <mesh filename="package://ob1_arm_description/meshes/arm/part_1.stl"/>
                 </geometry>
                 <material name="part_1_material">
@@ -474,5 +474,5 @@
                 <origin xyz="-0.0645733 -0.0670487 0.129369" rpy="-1.45249 0.81946 0.0866409" />
                 <geometry>
-                    <mesh filename="package://ob1_arm_description/meshes/part_2.stl"/>
+                    <mesh filename="package://ob1_arm_description/meshes/arm/part_2.stl"/>
                 </geometry>
                 <material name="part_2_material">
@@ -483,5 +483,5 @@
                 <origin xyz="-0.0645733 -0.0670487 0.129369" rpy="-1.45249 0.81946 0.0866409" />
                 <geometry>
-                    <mesh filename="package://ob1_arm_description/meshes/part_2.stl"/>
+                    <mesh filename="package://ob1_arm_description/meshes/arm/part_2.stl"/>
                 </geometry>
                 <material name="part_2_material">
@@ -492,5 +492,5 @@
                 <origin xyz="-0.0185543 0.0183829 0.0681824" rpy="-2.11035e-16 -0.0162981 -1.5708" />
                 <geometry>
-                    <mesh filename="package://ob1_arm_description/meshes/part_1.stl"/>
+                    <mesh filename="package://ob1_arm_description/meshes/arm/part_1.stl"/>
                 </geometry>
                 <material name="part_1_material">
@@ -501,5 +501,5 @@
                 <origin xyz="-0.0185543 0.0183829 0.0681824" rpy="-2.11035e-16 -0.0162981 -1.5708" />
                 <geometry>
-                    <mesh filename="package://ob1_arm_description/meshes/part_1.stl"/>
+                    <mesh filename="package://ob1_arm_description/meshes/arm/part_1.stl"/>
                 </geometry>
                 <material name="part_1_material">
@@ -510,5 +510,5 @@
                 <origin xyz="0.0988562 0.014795 0.216292" rpy="-1.5708 0.989151 -3.14159" />
                 <geometry>
-                    <mesh filename="package://ob1_arm_description/meshes/part_1.stl"/>
+                    <mesh filename="package://ob1_arm_description/meshes/arm/part_1.stl"/>
                 </geometry>
                 <material name="part_1_material">
@@ -519,5 +519,5 @@
                 <origin xyz="0.0988562 0.014795 0.216292" rpy="-1.5708 0.989151 -3.14159" />
                 <geometry>
-                    <mesh filename="package://ob1_arm_description/meshes/part_1.stl"/>
+                    <mesh filename="package://ob1_arm_description/meshes/arm/part_1.stl"/>
                 </geometry>
                 <material name="part_1_material">
@@ -528,5 +528,5 @@
                 <origin xyz="-0.0793646 0.0346641 0.226122" rpy="-1.60498 1.07372 -0.0300488" />
                 <geometry>
-                    <mesh filename="package://ob1_arm_description/meshes/part_2.stl"/>
+                    <mesh filename="package://ob1_arm_description/meshes/arm/part_2.stl"/>
                 </geometry>
                 <material name="part_2_material">
@@ -537,5 +537,5 @@
                 <origin xyz="-0.0793646 0.0346641 0.226122" rpy="-1.60498 1.07372 -0.0300488" />
                 <geometry>
-                    <mesh filename="package://ob1_arm_description/meshes/part_2.stl"/>
+                    <mesh filename="package://ob1_arm_description/meshes/arm/part_2.stl"/>
                 </geometry>
                 <material name="part_2_material">
@@ -546,5 +546,5 @@
                 <origin xyz="-0.0830985 -0.0669066 0.183302" rpy="-1.42635 0.976747 0.119958" />
                 <geometry>
-                    <mesh filename="package://ob1_arm_description/meshes/part_4.stl"/>
+                    <mesh filename="package://ob1_arm_description/meshes/arm/part_4.stl"/>
                 </geometry>
                 <material name="part_4_material">
@@ -555,5 +555,5 @@
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