Commit message: Added kinpy for faster fk calcualtions and tested kinpy ik calcualtions (not that accurate), generated much larger reachability point space (2 million points), refactor some code and minor improvements to testcases

File: ob1_arm_description/urdf/ob1_arm.xacro (robot description, xacro)
@@ -438,5 +438,5 @@
         <child link="${prefix}_forearm_link" />
         <axis xyz="0 0 1"/>
-        <limit effort="1" velocity="20" lower="-3.14" upper="3.14"/>
+        <limit effort="1" velocity="20" lower="-1.5787" upper="1.5787"/>
         <joint_properties friction="0.0"/>
         <dynamics D="1" K="7000" mu_coulomb="0" mu_viscous="16" damping="0.003" friction="0.0"/>
@@ -456,5 +456,5 @@
         <child link="${prefix}_arm_link" />
         <axis xyz="0 0 1"/>
-        <limit effort="1" velocity="20" lower="-3.14" upper="3.14"/>
+        <limit effort="1" velocity="20" lower="-1.5787" upper="1.5787"/>
         <joint_properties friction="0.0"/>
         <dynamics D="1" K="7000" mu_coulomb="0" mu_viscous="16" damping="0.003" friction="0.0"/>
@@ -465,5 +465,5 @@
         <child link="${prefix}_shoulder_link" />
         <axis xyz="0 0 1"/>
-        <limit effort="1" velocity="20" lower="-3.14" upper="3.14"/>
+        <limit effort="1" velocity="20" lower="-1.5787" upper="1.5787"/>
         <joint_properties friction="0.0"/>
         <dynamics D="1" K="7000" mu_coulomb="0" mu_viscous="16" damping="0.003" friction="0.0"/>
