Commit message: moved eef to tip of gripper between both claws, did this by adding 'imaginary and fixed eef link'

File: ob1_arm_description/urdf/gripper.xacro (robot description, xacro)
@@ -308,5 +308,5 @@
         <origin xyz="0 0 0" rpy="0 0 0"/>
         <mass value="0" />
-        <inertia ixx="0" ixy="0"  ixz="0" iyy="0" iyz="0" izz="0" />
+        <inertia ixx="0" ixy="0"  ixz="0" iyy="0" iyz="0" izz="0" />eef
         </inertial>
         </link>
@@ -329,4 +329,16 @@
         <dynamics D="1" K="7000" mu_coulomb="0" mu_viscous="16" damping="0.003" friction="0.0"/>
         </joint>
+        <link name="${prefix}_eef_link">
+            <inertial>
+                <origin xyz="0 0 0" rpy="0 0 0"/>
+                <mass value="0" />
+                <inertia ixx="0" ixy="0"  ixz="0" iyy="0" iyz="0" izz="0" />
+            </inertial>
+        </link>
+        <joint name="${prefix}_gripper_eef_link" type="fixed">
+            <origin xyz="0 0 -0.11" rpy="0 0 0" />
+            <parent link="${prefix}_gripper_base_link" />
+            <child link="${prefix}_eef_link" />
+        </joint>
     </xacro:macro>
 </robot>

File: ob1_arm_description/urdf/gripper_no_collision.xacro (robot description, xacro)
@@ -329,4 +329,16 @@
         <dynamics D="1" K="7000" mu_coulomb="0" mu_viscous="16" damping="0.003" friction="0.0"/>
         </joint>
+        <link name="${prefix}_eef_link">
+            <inertial>
+                <origin xyz="0 0 0" rpy="0 0 0"/>
+                <mass value="0" />
+                <inertia ixx="0" ixy="0"  ixz="0" iyy="0" iyz="0" izz="0" />
+            </inertial>
+        </link>
+        <joint name="${prefix}_gripper_eef_link" type="fixed">
+            <origin xyz="0 0 -0.11" rpy="0 0 0" />
+            <parent link="${prefix}_gripper_base_link" />
+            <child link="${prefix}_eef_link" />
+        </joint>
     </xacro:macro>
 </robot>

File: ob1_arm_description/urdf/main.urdf (robot description, URDF)
Before this commit: robot robot, 8 links, 7 joints
Links:
- added link ob1_arm_eef_link, mass 0
Joints:
- added joint ob1_arm_gripper_eef_link: type fixed, parent ob1_arm_gripper_base_link, child ob1_arm_eef_link, origin xyz=0 0 -0.11 rpy=0 0 0

Commit message: relaxed ik submodule and package configured

File: ob1_arm_description/urdf/gripper.xacro (robot description, xacro)
@@ -336,5 +336,5 @@
             </inertial>
         </link>
-        <joint name="${prefix}_gripper_eef_link" type="fixed">
+        <joint name="${prefix}_gripper_eef_joint" type="fixed">
             <origin xyz="0 0 -0.11" rpy="0 0 0" />
             <parent link="${prefix}_gripper_base_link" />

File: ob1_arm_description/urdf/gripper_no_collision.xacro (robot description, xacro)
@@ -336,5 +336,5 @@
             </inertial>
         </link>
-        <joint name="${prefix}_gripper_eef_link" type="fixed">
+        <joint name="${prefix}_gripper_eef_joint" type="fixed">
             <origin xyz="0 0 -0.11" rpy="0 0 0" />
             <parent link="${prefix}_gripper_base_link" />

File: ob1_arm_description/urdf/main.urdf (robot description, URDF)
Before this commit: robot robot, 9 links, 8 joints
Joints:
- removed joint ob1_arm_gripper_eef_link
- added joint ob1_arm_gripper_eef_joint: type fixed, parent ob1_arm_gripper_base_link, child ob1_arm_eef_link, origin xyz=0 0 -0.11 rpy=0 0 0
