Commit message: sixth joint and some test case modifications for position/pose testing as well as modifiying go position in arm commander

File: ob1_arm_description/urdf/main.xacro (robot description, xacro)
@@ -24,5 +24,5 @@
     <joint name="base" type="fixed">
         <parent link="world" />
-        <child link="${prefix}_base_link" />
+        <child link="${prefix}_fixed_base_link" />
     </joint>
 </robot>

File: ob1_arm_description/urdf/ob1_arm.xacro (robot description, xacro)
@@ -2,4 +2,11 @@
 <robot xmlns:xacro="http://www.ros.org/wiki/xacro" name="robot">
     <xacro:macro name="arm" params="prefix">
+        <link name="${prefix}_fixed_base_link">
+            <inertial>
+                <origin xyz="0 0 0" rpy="0 0 0"/>
+                <mass value="0" />
+                <inertia ixx="0" ixy="0"  ixz="0" iyy="0" iyz="0" izz="0" />
+            </inertial>
+        </link>
         <link name="${prefix}_base_link">
         <visual>
@@ -469,4 +476,13 @@
         <dynamics D="1" K="7000" mu_coulomb="0" mu_viscous="16" damping="0.003" friction="0.0"/>
         </joint>
+        <joint name="${prefix}_fixed_base_joint" type="revolute">
+        <origin xyz="0 0 0" rpy="0 0 0" />
+        <parent link="${prefix}_fixed_base_link" />
+        <child link="${prefix}_base_link" />
+        <axis xyz="0 0 1"/>
+        <limit effort="1" velocity="20" lower="-3.14" upper="3.14"/>
+        <joint_properties friction="0.0"/>
+        <dynamics D="1" K="7000" mu_coulomb="0" mu_viscous="16" damping="0.003" friction="0.0"/>
+        </joint>
     </xacro:macro>
 </robot>

Commit message: Revert "Merge pull request #8 from UBC-OpenRobotics/sixth_joint_urdf"
This reverts commit 60220c8fabf89ec6d4f9765121289dd51f09c289, reversing
changes made to bcc7858c849d4ad9a26ab226ade1542fb6a17119.

File: ob1_arm_description/urdf/main.xacro (robot description, xacro)
@@ -24,5 +24,5 @@
     <joint name="base" type="fixed">
         <parent link="world" />
-        <child link="${prefix}_fixed_base_link" />
+        <child link="${prefix}_base_link" />
     </joint>
 </robot>

File: ob1_arm_description/urdf/ob1_arm.xacro (robot description, xacro)
@@ -2,11 +2,4 @@
 <robot xmlns:xacro="http://www.ros.org/wiki/xacro" name="robot">
     <xacro:macro name="arm" params="prefix">
-        <link name="${prefix}_fixed_base_link">
-            <inertial>
-                <origin xyz="0 0 0" rpy="0 0 0"/>
-                <mass value="0" />
-                <inertia ixx="0" ixy="0"  ixz="0" iyy="0" iyz="0" izz="0" />
-            </inertial>
-        </link>
         <link name="${prefix}_base_link">
         <visual>
@@ -476,13 +469,4 @@
         <dynamics D="1" K="7000" mu_coulomb="0" mu_viscous="16" damping="0.003" friction="0.0"/>
         </joint>
-        <joint name="${prefix}_fixed_base_joint" type="revolute">
-        <origin xyz="0 0 0" rpy="0 0 0" />
-        <parent link="${prefix}_fixed_base_link" />
-        <child link="${prefix}_base_link" />
-        <axis xyz="0 0 1"/>
-        <limit effort="1" velocity="20" lower="-3.14" upper="3.14"/>
-        <joint_properties friction="0.0"/>
-        <dynamics D="1" K="7000" mu_coulomb="0" mu_viscous="16" damping="0.003" friction="0.0"/>
-        </joint>
     </xacro:macro>
 </robot>
