Commit message: created python packages for arm_commander, and util in ob1_arm_control rospkg, refactored pytest test cases, added new fixtures and conftest.py and pytest.ini for test/fixture configurations. Reconstructed main.urdf with latest main.xacro

File: ob1_arm_description/urdf/main.urdf (robot description, URDF)
Before this commit: robot robot, 9 links, 8 joints
Links:
- added link ob1_arm_fixed_base_link, mass 0
- added link world
Joints:
- added joint base: type fixed, parent world, child ob1_arm_fixed_base_link
- added joint ob1_arm_fixed_base_joint: type revolute, parent ob1_arm_fixed_base_link, child ob1_arm_base_link, origin xyz=0 0 0 rpy=0 0 0, axis 0 0 1, limit lower=-3.14 upper=3.14 effort=1 velocity=20
