Commit message: changes to mobile_base dimensions

File: ob1_arm_description/urdf/mobile_base.xacro (robot description, xacro)
@@ -37,4 +37,11 @@
   <!-- Hokuyo Laser scanner -->
   <!-- Macro for calculating inertia of cylinder -->
+  <!--
+  <link name="world"/>
+    <joint name="base" type="fixed">
+        <parent link="world" />
+        <child link="base_footprint" />
+    </joint>
+  -->
   <!-- BASE-FOOTPRINT -->
   <!-- base_footprint is a fictitious link(frame) that is on the ground right below base_link origin -->
@@ -56,5 +63,5 @@
   </gazebo>
   <joint name="base_footprint_joint" type="fixed">
-    <origin rpy="0 0 0" xyz="0 0 0.04"/>
+    <origin rpy="0 0 0" xyz="0 0 0.09319"/> <!--changed z coordinate-->
     <parent link="base_footprint"/>
     <child link="base_link"/>
@@ -72,5 +79,5 @@
       <origin rpy="0 0 0" xyz="0 0 0"/>
       <geometry>
-        <cylinder length="0.02" radius="0.15"/>
+        <cylinder length="0.02" radius="0.15"/> <!--box: x = 0.5132 m ,y = 0.5132 m, z = 1.27976 m-->
       </geometry>
       <material name="${base_name}_White"/>
@@ -92,5 +99,5 @@
       <origin rpy="1.57079632679 0  0 " xyz="0 0 0"/>
       <geometry>
-        <cylinder length="0.02" radius="0.04"/>
+        <cylinder length="0.02" radius="0.09319"/> <!--changed radius-->
       </geometry>
       <material name="${base_name}_Red"/>
@@ -99,5 +106,5 @@
       <origin rpy="1.57079632679 0 0 " xyz="0 0 0"/>
       <geometry>
-        <cylinder length="0.02" radius="0.04"/>
+        <cylinder length="0.02" radius="0.09319"/> <!--changed radius-->
       </geometry>
     </collision>
@@ -120,5 +127,5 @@
     <parent link="base_link"/>
     <child link="front_right_wheel"/>
-    <origin rpy="0 0 0" xyz="0.0 0.15 0.0"/>
+    <origin rpy="0 0 0" xyz="0.0 0.308 0.0"/> <!--changed y coordinate-->
     <axis rpy="0  0" xyz="0 1 0"/>
     <limit effort="100" velocity="100"/>
@@ -139,5 +146,5 @@
       <origin rpy="1.57079632679 0  0 " xyz="0 0 0"/>
       <geometry>
-        <cylinder length="0.02" radius="0.04"/>
+        <cylinder length="0.02" radius="0.09319"/> <!--changed radius-->
       </geometry>
       <material name="${base_name}_Red"/>
@@ -146,5 +153,5 @@
       <origin rpy="1.57079632679 0 0 " xyz="0 0 0"/>
       <geometry>
-        <cylinder length="0.02" radius="0.04"/>
+        <cylinder length="0.02" radius="0.09319"/> <!--changed radius-->
       </geometry>
     </collision>
@@ -167,5 +174,5 @@
     <parent link="base_link"/>
     <child link="front_left_wheel"/>
-    <origin rpy="0 0 0" xyz="0.0 -0.15 0.0"/>
+    <origin rpy="0 0 0" xyz="0.0 -0.308 0.0"/> <!--changed y coordinate-->
     <axis rpy="0  0" xyz="0 1 0"/>
     <limit effort="100" velocity="100"/>
