Commit message: dynamic gripper urdf (2 joint apporximation) to attempt to grip objects

File: ob1_arm_description/onshape_to_robot/robot.urdf (robot description, URDF)
Before this commit: robot onshape, 6 links, 5 joints
Links:
- removed link arm_link
- removed link base_link
- removed link elbow_link
- removed link forearm_link
- removed link gripper_assembly_link
- removed link shoulder_link
- added link ${prefix}_arm_link, mass 0; collision mesh filename=package://ob1_arm_description/meshes/bicep_linkage_-_encode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; collision mesh filename=package://ob1_arm_description/meshes/bicep_linkage_-_motor.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
- added link ${prefix}_base_link, mass 0; collision mesh filename=package://ob1_arm_description/meshes/motor_front_support_-_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; collision mesh filename=package://ob1_arm_description/meshes/motor_mid_support_-_sh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
- added link ${prefix}_elbow_link, mass 0; collision mesh filename=package://ob1_arm_description/meshes/forearm_intermediate_p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; collision mesh filename=package://ob1_arm_description/meshes/forearm_motor_support.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
- added link ${prefix}_forearm_link, mass 0; collision mesh filename=package://ob1_arm_description/meshes/end_effector_plate.stl; collision mesh filename=package://ob1_arm_description/meshes/forearm_linkage_-_enco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
- added link ${prefix}_gripper_base_link, mass 0; collision mesh filename=package://ob1_arm_description/meshes/hk15328d_v5.stl; collision mesh filename=package://ob1_arm_description/meshes/hk15328d_v5.stl
- added link ${prefix}_lclaw_link, mass 0; collision mesh filename=package://ob1_arm_description/meshes/part_1_gripper_claw.stl; collision mesh filename=package://ob1_arm_description/meshes/part_2_gripper_claw.stl
- added link ${prefix}_rclaw_link, mass 0; collision mesh filename=package://ob1_arm_description/meshes/part_1_mirror_gripper_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; collision mesh filename=package://ob1_arm_description/meshes/part_2_mirror_gripper_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
- added link ${prefix}_shoulder_link, mass 0; collision mesh filename=package://ob1_arm_description/meshes/bicep_plate_-_real.stl; collision mesh filename=package://ob1_arm_description/meshes/bicep_y_motor.stl
Joints:
- removed joint arm_elbow_joint
- removed joint base_shoulder
- removed joint elbow_forearm_joint
- removed joint shoulder_arm
- removed joint wrist
- added joint ${prefix}_arm_elbow_joint: type revolute, parent ${prefix}_arm_link, child ${prefix}_elbow_link, origin xyz=-1.33227e-15 0.18 0.0475 rpy=1.5708 0.00373826 -5.38613e-15, axis 0 0 1, limit effort=1 velocity=20
- added joint ${prefix}_base_shoulder_joint: type revolute, parent ${prefix}_base_link, child ${prefix}_shoulder_link, origin xyz=8.1532e-17 0.0475 0.06 rpy=1.5708 -0.0134839 4.87562e-15, axis 0 0 1, limit effort=1 velocity=20
- added joint ${prefix}_elbow_forearm_joint: type revolute, parent ${prefix}_elbow_link, child ${prefix}_forearm_link, origin xyz=7.71952e-16 0.08285 -0.03115 rpy=1.5708 0.0729385 1.34977e-15, axis 0 0 1, limit effort=1 velocity=20
- added joint ${prefix}_forearm_gripper_joint: type revolute, parent ${prefix}_forearm_link, child ${prefix}_gripper_base_link, origin xyz=-2.46331e-16 -0.155 0.08285 rpy=-1.5708 0.278795 3.7292e-15, axis 0 0 1, limit effort=1 velocity=20
- added joint ${prefix}_gripper_lclaw_joint: type revolute, parent ${prefix}_gripper_base_link, child ${prefix}_lclaw_link, origin xyz=-0.04 0.008 -0.0535151 rpy=1.5708 -0.367452 -8.36952e-16, axis 0 0 1, limit effort=1 velocity=20
- added joint ${prefix}_gripper_rclaw_joint: type revolute, parent ${prefix}_{prefix}_gripper_base_link, child ${prefix}_rclaw_link, origin xyz=0.04 0.008 -0.0535151 rpy=1.5708 0.450222 1.06462e-15, axis 0 0 1, limit effort=1 velocity=20
- added joint ${prefix}_shoulder_arm_joint: type revolute, parent ${prefix}_shoulder_link, child ${prefix}_arm_link, origin xyz=2.90241e-16 0.15 -7.97973e-16 rpy=8.20328e-16 -1.37552e-14 -0.046259, axis 0 0 1, limit effort=1 velocity=20

File: ob1_arm_description/urdf/gripper.xacro (robot description, xacro)
@@ -2,299 +2,331 @@
 <robot xmlns:xacro="http://www.ros.org/wiki/xacro">
     <xacro:macro name="gripper" params="prefix">
-        <link name="${prefix}_gripper_assembly_link">
-            <visual>
-            <origin xyz="-0.04015 0.0144875 -0.0347028" rpy="-1.22013e-12 -1.55917 -1.5708" />
-            <geometry>
-            <mesh filename="package://ob1_arm_description/meshes/hk15328d_v5.stl"/>
-            </geometry>
-            <material name="hk15328d_v5_material">
-            <color rgba="0.392157 0.403922 0.384314 1.0"/>
-            </material>
-            </visual>
-            <collision>
-            <origin xyz="-0.04015 0.0144875 -0.0347028" rpy="-1.22013e-12 -1.55917 -1.5708" />
-            <geometry>
-            <mesh filename="package://ob1_arm_description/meshes/hk15328d_v5.stl"/>
-            </geometry>
-            <material name="hk15328d_v5_material">
-            <color rgba="0.392157 0.403922 0.384314 1.0"/>
-            </material>
-            </collision>
-            <visual>
-            <origin xyz="-0.0382059 -0.005 -0.100345" rpy="-1.34629e-14 -1.35876 1.29259e-14" />
-            <geometry>
-            <mesh filename="package://ob1_arm_description/meshes/part_2_gripper_claw.stl"/>
-            </geometry>
-            <material name="part_2_gripper_claw_material">
-            <color rgba="0.647059 0.647059 0.647059 1.0"/>
-            </material>
-            </visual>
-            <collision>
-            <origin xyz="-0.0382059 -0.005 -0.100345" rpy="-1.34629e-14 -1.35876 1.29259e-14" />
-            <geometry>
-            <mesh filename="package://ob1_arm_description/meshes/part_2_gripper_claw.stl"/>
-            </geometry>
-            <material name="part_2_gripper_claw_material">
-            <color rgba="0.647059 0.647059 0.647059 1.0"/>
-            </material>
-            </collision>
-            <visual>
-            <origin xyz="-0.0506217 -0.004 -0.0839523" rpy="3.14159 -2.35608e-17 -1.19404e-17" />
-            <geometry>
-            <mesh filename="package://ob1_arm_description/meshes/part_3_gripper_claw.stl"/>
-            </geometry>
-            <material name="part_3_gripper_claw_material">
-            <color rgba="0.231373 0.380392 0.705882 1.0"/>
-            </material>
-            </visual>
-            <collision>
-            <origin xyz="-0.0506217 -0.004 -0.0839523" rpy="3.14159 -2.35608e-17 -1.19404e-17" />
-            <geometry>
-            <mesh filename="package://ob1_arm_description/meshes/part_3_gripper_claw.stl"/>
-            </geometry>
-            <material name="part_3_gripper_claw_material">
-            <color rgba="0.231373 0.380392 0.705882 1.0"/>
-            </material>
-            </collision>
-            <visual>
-            <origin xyz="-0.0182314 -0.029 -0.0656435" rpy="3.14159 -0.039707 1.67593e-14" />
-            <geometry>
-            <mesh filename="package://ob1_arm_description/meshes/part_1_gripper_claw.stl"/>
-            </geometry>
-            <material name="part_1_gripper_claw_material">
-            <color rgba="0.615686 0.811765 0.929412 1.0"/>
-            </material>
-            </visual>
-            <collision>
-            <origin xyz="-0.0182314 -0.029 -0.0656435" rpy="3.14159 -0.039707 1.67593e-14" />
-            <geometry>
-            <mesh filename="package://ob1_arm_description/meshes/part_1_gripper_claw.stl"/>
-            </geometry>
-            <material name="part_1_gripper_claw_material">
-            <color rgba="0.615686 0.811765 0.929412 1.0"/>
-            </material>
-            </collision>
-            <visual>
-            <origin xyz="0.0209978 -0.029 -0.0626659" rpy="3.14159 0.073635 1.24744e-14" />
-            <geometry>
-            <mesh filename="package://ob1_arm_description/meshes/part_1_mirror_gripper_claw.stl"/>
-            </geometry>
-            <material name="part_1_mirror_gripper_claw_material">
-            <color rgba="0.615686 0.811765 0.929412 1.0"/>
-            </material>
-            </visual>
-            <collision>
-            <origin xyz="0.0209978 -0.029 -0.0626659" rpy="3.14159 0.073635 1.24744e-14" />
-            <geometry>
-            <mesh filename="package://ob1_arm_description/meshes/part_1_mirror_gripper_claw.stl"/>
-            </geometry>
-            <material name="part_1_mirror_gripper_claw_material">
-            <color rgba="0.615686 0.811765 0.929412 1.0"/>
-            </material>
-            </collision>
-            <visual>
-            <origin xyz="0.04015 0.0144875 -0.0347028" rpy="-5.18357e-13 1.55917 1.5708" />
-            <geometry>
-            <mesh filename="package://ob1_arm_description/meshes/hk15328d_v5.stl"/>
-            </geometry>
-            <material name="hk15328d_v5_material">
-            <color rgba="0.392157 0.403922 0.384314 1.0"/>
-            </material>
-            </visual>
-            <collision>
-            <origin xyz="0.04015 0.0144875 -0.0347028" rpy="-5.18357e-13 1.55917 1.5708" />
-            <geometry>
-            <mesh filename="package://ob1_arm_description/meshes/hk15328d_v5.stl"/>
-            </geometry>
-            <material name="hk15328d_v5_material">
-            <color rgba="0.392157 0.403922 0.384314 1.0"/>
-            </material>
-            </collision>
-            <visual>
-            <origin xyz="0.04 0.024 -0.0535151" rpy="-2.85212e-15 -2.06882e-17 -3.79317e-17" />
-            <geometry>
-            <mesh filename="package://ob1_arm_description/meshes/spur_gear_(36_teeth).stl"/>
-            </geometry>
-            <material name="spur_gear_(36_teeth)_material">
-            <color rgba="0.647059 0.647059 0.647059 1.0"/>
-            </material>
-            </visual>
-            <collision>
-            <origin xyz="0.04 0.024 -0.0535151" rpy="-2.85212e-15 -2.06882e-17 -3.79317e-17" />
-            <geometry>
-            <mesh filename="package://ob1_arm_description/meshes/spur_gear_(36_teeth).stl"/>
-            </geometry>
-            <material name="spur_gear_(36_teeth)_material">
-            <color rgba="0.647059 0.647059 0.647059 1.0"/>
-            </material>
-            </collision>
-            <visual>
-            <origin xyz="2.77556e-16 1.73472e-18 8.88178e-16" rpy="3.14159 -4.38952e-18 -9.64226e-17" />
-            <geometry>
-            <mesh filename="package://ob1_arm_description/meshes/part_2_gripper.stl"/>
-            </geometry>
-            <material name="part_2_gripper_material">
-            <color rgba="0.917647 0.917647 0.917647 1.0"/>
-            </material>
-            </visual>
-            <collision>
-            <origin xyz="2.77556e-16 1.73472e-18 8.88178e-16" rpy="3.14159 -4.38952e-18 -9.64226e-17" />
-            <geometry>
-            <mesh filename="package://ob1_arm_description/meshes/part_2_gripper.stl"/>
-            </geometry>
-            <material name="part_2_gripper_material">
-            <color rgba="0.917647 0.917647 0.917647 1.0"/>
-            </material>
-            </collision>
-            <visual>
-            <origin xyz="0 1.73472e-18 0" rpy="3.14159 -9.58512e-18 1.23104e-17" />
-            <geometry>
-            <mesh filename="package://ob1_arm_description/meshes/part_1_gripper.stl"/>
-            </geometry>
-            <material name="part_1_gripper_material">
-            <color rgba="0.615686 0.811765 0.929412 1.0"/>
-            </material>
-            </visual>
-            <collision>
-            <origin xyz="0 1.73472e-18 0" rpy="3.14159 -9.58512e-18 1.23104e-17" />
-            <geometry>
-            <mesh filename="package://ob1_arm_description/meshes/part_1_gripper.stl"/>
-            </geometry>
-            <material name="part_1_gripper_material">
-            <color rgba="0.615686 0.811765 0.929412 1.0"/>
-            </material>
-            </collision>
-            <visual>
-            <origin xyz="-0.04015 0.0144875 -0.0347028" rpy="-1.54483 -1.1065 -0.02322" />
-            <geometry>
-            <mesh filename="package://ob1_arm_description/meshes/hk15328d_v5.stl"/>
-            </geometry>
-            <material name="hk15328d_v5_material">
-            <color rgba="0.952941 0.796078 0.486275 1.0"/>
-            </material>
-            </visual>
-            <collision>
-            <origin xyz="-0.04015 0.0144875 -0.0347028" rpy="-1.54483 -1.1065 -0.02322" />
-            <geometry>
-            <mesh filename="package://ob1_arm_description/meshes/hk15328d_v5.stl"/>
-            </geometry>
-            <material name="hk15328d_v5_material">
-            <color rgba="0.952941 0.796078 0.486275 1.0"/>
-            </material>
-            </collision>
-            <visual>
-            <origin xyz="-0.04 0.019 -0.0535151" rpy="3.14159 -0.174533 7.48986e-17" />
-            <geometry>
-            <mesh filename="package://ob1_arm_description/meshes/spur_gear_(36_teeth).stl"/>
-            </geometry>
-            <material name="spur_gear_(36_teeth)_material">
-            <color rgba="0.647059 0.647059 0.647059 1.0"/>
-            </material>
-            </visual>
-            <collision>
-            <origin xyz="-0.04 0.019 -0.0535151" rpy="3.14159 -0.174533 7.48986e-17" />
-            <geometry>
-            <mesh filename="package://ob1_arm_description/meshes/spur_gear_(36_teeth).stl"/>
-            </geometry>
-            <material name="spur_gear_(36_teeth)_material">
-            <color rgba="0.647059 0.647059 0.647059 1.0"/>
-            </material>
-            </collision>
-            <visual>
-            <origin xyz="0.04015 0.0144875 -0.0347028" rpy="-1.44532 -1.47775 -0.124935" />
-            <geometry>
-            <mesh filename="package://ob1_arm_description/meshes/hk15328d_v5.stl"/>
-            </geometry>
-            <material name="hk15328d_v5_material">
-            <color rgba="0.952941 0.796078 0.486275 1.0"/>
-            </material>
-            </visual>
-            <collision>
-            <origin xyz="0.04015 0.0144875 -0.0347028" rpy="-1.44532 -1.47775 -0.124935" />
-            <geometry>
-            <mesh filename="package://ob1_arm_description/meshes/hk15328d_v5.stl"/>
-            </geometry>
-            <material name="hk15328d_v5_material">
-            <color rgba="0.952941 0.796078 0.486275 1.0"/>
-            </material>
-            </collision>
-            <visual>
-            <origin xyz="0.0391983 -0.005 -0.0996329" rpy="-1.18193e-14 1.32595 4.07848e-14" />
-            <geometry>
-            <mesh filename="package://ob1_arm_description/meshes/part_2_mirror_gripper_claw.stl"/>
-            </geometry>
-            <material name="part_2_mirror_gripper_claw_material">
-            <color rgba="0.647059 0.647059 0.647059 1.0"/>
-            </material>
-            </visual>
-            <collision>
-            <origin xyz="0.0391983 -0.005 -0.0996329" rpy="-1.18193e-14 1.32595 4.07848e-14" />
-            <geometry>
-            <mesh filename="package://ob1_arm_description/meshes/part_2_mirror_gripper_claw.stl"/>
-            </geometry>
-            <material name="part_2_mirror_gripper_claw_material">
-            <color rgba="0.647059 0.647059 0.647059 1.0"/>
-            </material>
-            </collision>
-            <visual>
-            <origin xyz="0.0506217 -0.004 -0.0839523" rpy="3.14159 -2.35608e-17 -1.19404e-17" />
-            <geometry>
-            <mesh filename="package://ob1_arm_description/meshes/part_3_mirror_gripper_claw.stl"/>
-            </geometry>
-            <material name="part_3_mirror_gripper_claw_material">
-            <color rgba="0.231373 0.380392 0.705882 1.0"/>
-            </material>
-            </visual>
-            <collision>
-            <origin xyz="0.0506217 -0.004 -0.0839523" rpy="3.14159 -2.35608e-17 -1.19404e-17" />
-            <geometry>
-            <mesh filename="package://ob1_arm_description/meshes/part_3_mirror_gripper_claw.stl"/>
-            </geometry>
-            <material name="part_3_mirror_gripper_claw_material">
-            <color rgba="0.231373 0.380392 0.705882 1.0"/>
-            </material>
-            </collision>
-            <visual>
-            <origin xyz="0.04015 0.0239869 -0.0345924" rpy="0.125472 -1.47775 -0.124935" />
-            <geometry>
-            <mesh filename="package://ob1_arm_description/meshes/spur_gear_(16_teeth).stl"/>
-            </geometry>
-            <material name="spur_gear_(16_teeth)_material">
-            <color rgba="0.615686 0.811765 0.929412 1.0"/>
-            </material>
-            </visual>
-            <collision>
-            <origin xyz="0.04015 0.0239869 -0.0345924" rpy="0.125472 -1.47775 -0.124935" />
-            <geometry>
-            <mesh filename="package://ob1_arm_description/meshes/spur_gear_(16_teeth).stl"/>
-            </geometry>
-            <material name="spur_gear_(16_teeth)_material">
-            <color rgba="0.615686 0.811765 0.929412 1.0"/>
-            </material>
-            </collision>
-            <visual>
-            <origin xyz="-0.04015 0.0239869 -0.0345924" rpy="0.0259681 -1.1065 -0.02322" />
-            <geometry>
-            <mesh filename="package://ob1_arm_description/meshes/spur_gear_(16_teeth).stl"/>
-            </geometry>
-            <material name="spur_gear_(16_teeth)_material">
-            <color rgba="0.615686 0.811765 0.929412 1.0"/>
-            </material>
-            </visual>
-            <collision>
-            <origin xyz="-0.04015 0.0239869 -0.0345924" rpy="0.0259681 -1.1065 -0.02322" />
-            <geometry>
-            <mesh filename="package://ob1_arm_description/meshes/spur_gear_(16_teeth).stl"/>
-            </geometry>
-            <material name="spur_gear_(16_teeth)_material">
-            <color rgba="0.615686 0.811765 0.929412 1.0"/>
-            </material>
-            </collision>
-            <inertial>
-            <origin xyz="0 0 0" rpy="0 0 0"/>
-            <mass value="0" />
-            <inertia ixx="0" ixy="0"  ixz="0" iyy="0" iyz="0" izz="0" />
-            </inertial>
+        <link name="${prefix}_gripper_base_link">
+        <visual>
+        <origin xyz="-0.04015 0.0144875 -0.0347028" rpy="-1.31921 -1.52407 -0.251324" />
+        <geometry>
+        <mesh filename="package://ob1_arm_description/meshes/hk15328d_v5.stl"/>
+        </geometry>
+        <material name="hk15328d_v5_material">
+        <color rgba="0.952941 0.796078 0.486275 1.0"/>
+        </material>
+        </visual>
+        <collision>
+        <origin xyz="-0.04015 0.0144875 -0.0347028" rpy="-1.31921 -1.52407 -0.251324" />
+        <geometry>
+        <mesh filename="package://ob1_arm_description/meshes/hk15328d_v5.stl"/>
+        </geometry>
+        <material name="hk15328d_v5_material">
+        <color rgba="0.952941 0.796078 0.486275 1.0"/>
+        </material>
+        </collision>
+        <visual>
+        <origin xyz="-0.04015 0.0239869 -0.0345924" rpy="0.251587 -1.52407 -0.251324" />
+        <geometry>
+        <mesh filename="package://ob1_arm_description/meshes/spur_gear_(16_teeth).stl"/>
+        </geometry>
+        <material name="spur_gear_(16_teeth)_material">
+        <color rgba="0.615686 0.811765 0.929412 1.0"/>
+        </material>
+        </visual>
+        <collision>
+        <origin xyz="-0.04015 0.0239869 -0.0345924" rpy="0.251587 -1.52407 -0.251324" />
+        <geometry>
+        <mesh filename="package://ob1_arm_description/meshes/spur_gear_(16_teeth).stl"/>
+        </geometry>
+        <material name="spur_gear_(16_teeth)_material">
+        <color rgba="0.615686 0.811765 0.929412 1.0"/>
+        </material>
+        </collision>
+        <visual>
+        <origin xyz="-0.04 0.019 -0.0535151" rpy="-3.14159 -0.174533 4.4254e-17" />
+        <geometry>
+        <mesh filename="package://ob1_arm_description/meshes/spur_gear_(36_teeth).stl"/>
+        </geometry>
+        <material name="spur_gear_(36_teeth)_material">
+        <color rgba="0.647059 0.647059 0.647059 1.0"/>
+        </material>
+        </visual>
+        <collision>
+        <origin xyz="-0.04 0.019 -0.0535151" rpy="-3.14159 -0.174533 4.4254e-17" />
+        <geometry>
+        <mesh filename="package://ob1_arm_description/meshes/spur_gear_(36_teeth).stl"/>
+        </geometry>
+        <material name="spur_gear_(36_teeth)_material">
+        <color rgba="0.647059 0.647059 0.647059 1.0"/>
+        </material>
+        </collision>
+        <visual>
+        <origin xyz="6.93889e-18 -8.67362e-19 -1.77636e-15" rpy="-3.14159 1.01857e-14 5.54818e-17" />
+        <geometry>
+        <mesh filename="package://ob1_arm_description/meshes/part_2_gripper.stl"/>
+        </geometry>
+        <material name="part_2_gripper_material">
+        <color rgba="0.917647 0.917647 0.917647 1.0"/>
+        </material>
+        </visual>
+        <collision>
+        <origin xyz="6.93889e-18 -8.67362e-19 -1.77636e-15" rpy="-3.14159 1.01857e-14 5.54818e-17" />
+        <geometry>
+        <mesh filename="package://ob1_arm_description/meshes/part_2_gripper.stl"/>
+        </geometry>
+        <material name="part_2_gripper_material">
+        <color rgba="0.917647 0.917647 0.917647 1.0"/>
+        </material>
+        </collision>
+        <visual>
+        <origin xyz="0.04015 0.0239869 -0.0345924" rpy="3.10536 -1.244 -3.10728" />
+        <geometry>
+        <mesh filename="package://ob1_arm_description/meshes/spur_gear_(16_teeth).stl"/>
+        </geometry>
+        <material name="spur_gear_(16_teeth)_material">
+        <color rgba="0.615686 0.811765 0.929412 1.0"/>
+        </material>
+        </visual>
+        <collision>
+        <origin xyz="0.04015 0.0239869 -0.0345924" rpy="3.10536 -1.244 -3.10728" />
+        <geometry>
+        <mesh filename="package://ob1_arm_description/meshes/spur_gear_(16_teeth).stl"/>
+        </geometry>
+        <material name="spur_gear_(16_teeth)_material">
+        <color rgba="0.615686 0.811765 0.929412 1.0"/>
+        </material>
+        </collision>
+        <visual>
+        <origin xyz="0.04 0.024 -0.0535151" rpy="1.10827e-14 1.0192e-14 1.02561e-16" />
+        <geometry>
+        <mesh filename="package://ob1_arm_description/meshes/spur_gear_(36_teeth).stl"/>
+        </geometry>
+        <material name="spur_gear_(36_teeth)_material">
+        <color rgba="0.647059 0.647059 0.647059 1.0"/>
+        </material>
+        </visual>
+        <collision>
+        <origin xyz="0.04 0.024 -0.0535151" rpy="1.10827e-14 1.0192e-14 1.02561e-16" />
+        <geometry>
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