Commit message: refactored and added better comments to test cases, ran joint, position, and pose tests to confirm that the 6th joint improves planning success rate, and ran pick sphere tests

File: ob1_arm_moveit_config/config/gazebo_robot.urdf (robot description, URDF)
Before this commit: robot robot, 11 links, 10 joints
Joints:
- removed joint ob1_arm_gripper_eef_link
- added joint ob1_arm_gripper_eef_joint: type fixed, parent ob1_arm_gripper_base_link, child ob1_arm_eef_link, origin xyz=0 0 -0.11 rpy=0 0 0
