Commit message: refactored moveit config packages into one sub directory, and added back the old configuration to keep track of it (5dof configuration).

File: moveit_configs/dof_5_moveit_config/config/gazebo_robot.urdf (robot description, URDF)
Before this commit: robot robot, 11 links, 10 joints
Links:
- removed link ob1_arm_fixed_base_link
Joints:
- removed joint ob1_arm_fixed_base_joint
- removed joint ob1_arm_gripper_eef_link
- added joint ob1_arm_gripper_eef_joint: type fixed, parent ob1_arm_gripper_base_link, child ob1_arm_eef_link, origin xyz=0 0 -0.11 rpy=0 0 0
- joint base: child ob1_arm_fixed_base_link -> ob1_arm_base_link
