Commit message: created ik fast plugin for ob1_arm urdf, refactored ik solvers into subdirectory,test case changes

File: ik_solvers/matlab_ik/main.urdf (robot description, URDF)
Before this commit: robot robot, 8 links, 7 joints
Links:
- removed link ob1_arm_lclaw_link
- removed link ob1_arm_rclaw_link
- added link ob1_arm_eef_link, mass 0
- added link ob1_arm_fixed_base_link, mass 0
- link ob1_arm_arm_link: geometry collision mesh filename=package://ob1_arm_description/meshes/bicep_linkage_-_encode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; collision mesh filename=package://ob1_arm_description/meshes/bicep_linkage_-_motor.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
- link ob1_arm_base_link: geometry collision mesh filename=package://ob1_arm_description/meshes/motor_front_support_-_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; collision mesh filename=package://ob1_arm_description/meshes/motor_mid_support_-_sh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
- link ob1_arm_elbow_link: geometry collision mesh filename=package://ob1_arm_description/meshes/forearm_intermediate_p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; collision mesh filename=package://ob1_arm_description/meshes/forearm_motor_support.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
- link ob1_arm_forearm_link: geometry collision mesh filename=package://ob1_arm_description/meshes/end_effector_plate.stl; collision mesh filename=package://ob1_arm_description/meshes/forearm_linkage_-_enco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
- link ob1_arm_gripper_base_link: geometry collision mesh filename=package://ob1_arm_description/meshes/hk15328d_v5.stl; collision mesh filename=package://ob1_arm_description/meshes/hk15328d_v5.stl
- link ob1_arm_shoulder_link: geometry collision mesh filename=package://ob1_arm_description/meshes/bicep_plate_-_real.stl; collision mesh filename=package://ob1_arm_description/meshes/bicep_y_motor.stl
Joints:
- removed joint ob1_arm_gripper_lclaw_joint
- removed joint ob1_arm_gripper_rclaw_joint
- added joint ob1_arm_fixed_base_joint: type revolute, parent ob1_arm_fixed_base_link, child ob1_arm_base_link, origin xyz=0 0 0 rpy=0 0 0, axis 0 0 1, limit lower=-3.14 upper=3.14 effort=1 velocity=20
- added joint ob1_arm_gripper_eef_joint: type fixed, parent ob1_arm_gripper_base_link, child ob1_arm_eef_link, origin xyz=0 0 -0.11 rpy=0 0 0
- joint ob1_arm_arm_elbow_joint: origin xyz=0 0.18 0.0475 rpy=1.5708 0.00373826 0 -> xyz=-1.33227e-15 0.18 0.0475 rpy=1.5708 0.00373826 -5.38613e-15
- joint ob1_arm_base_shoulder_joint: origin xyz=0 0.0475 0.06 rpy=1.5708 -0.0134839 0 -> xyz=8.1532e-17 0.0475 0.06 rpy=1.5708 -0.0134839 4.87562e-15
- joint ob1_arm_elbow_forearm_joint: origin xyz=0 0.08285 -0.03115 rpy=1.5708 0.0729385 0 -> xyz=7.71952e-16 0.08285 -0.03115 rpy=1.5708 0.0729385 1.34977e-15
- joint ob1_arm_forearm_gripper_joint: origin xyz=0 -0.155 0.08285 rpy=-1.5708 0.278795 0 -> xyz=-2.46331e-16 -0.155 0.08285 rpy=-1.5708 0.278795 3.7292e-15
- joint ob1_arm_shoulder_arm_joint: origin xyz=0 0.15 0 rpy=0 0 -0.046259 -> xyz=2.90241e-16 0.15 -7.97973e-16 rpy=8.20328e-16 -1.37552e-14 -0.046259

File: ik_solvers/robot_arm_ikfast_plugin/temp/main.urdf (robot description, URDF)
Before this commit: robot robot, 9 links, 8 joints
Links:
- removed link ob1_arm_lclaw_link
- removed link ob1_arm_rclaw_link
- added link ob1_arm_fixed_base_link, mass 0
- link ob1_arm_arm_link: geometry collision mesh filename=package://ob1_arm_description/meshes/bicep_linkage_-_encode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; collision mesh filename=package://ob1_arm_description/meshes/bicep_linkage_-_motor.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
- link ob1_arm_base_link: geometry collision mesh filename=package://ob1_arm_description/meshes/motor_front_support_-_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; collision mesh filename=package://ob1_arm_description/meshes/motor_mid_support_-_sh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
- link ob1_arm_elbow_link: geometry collision mesh filename=package://ob1_arm_description/meshes/forearm_intermediate_p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; collision mesh filename=package://ob1_arm_description/meshes/forearm_motor_support.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
- link ob1_arm_forearm_link: geometry collision mesh filename=package://ob1_arm_description/meshes/end_effector_plate.stl; collision mesh filename=package://ob1_arm_description/meshes/forearm_linkage_-_enco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
- link ob1_arm_gripper_base_link: geometry collision mesh filename=package://ob1_arm_description/meshes/hk15328d_v5.stl; collision mesh filename=package://ob1_arm_description/meshes/hk15328d_v5.stl
- link ob1_arm_shoulder_link: geometry collision mesh filename=package://ob1_arm_description/meshes/bicep_plate_-_real.stl; collision mesh filename=package://ob1_arm_description/meshes/bicep_y_motor.stl
Joints:
- removed joint ob1_arm_gripper_lclaw_joint
- removed joint ob1_arm_gripper_rclaw_joint
- added joint ob1_arm_fixed_base_joint: type revolute, parent ob1_arm_fixed_base_link, child ob1_arm_base_link, origin xyz=0 0 0 rpy=0 0 0, axis 0 0 1, limit lower=-3.14 upper=3.14 effort=1 velocity=20

File: ob1_arm_description/urdf/main.urdf (robot description, URDF)
Before this commit: robot robot, 11 links, 10 joints
Links:
- removed link ob1_arm_lclaw_link
- removed link ob1_arm_rclaw_link
- removed link world
Joints:
- removed joint base
- removed joint ob1_arm_gripper_lclaw_joint
- removed joint ob1_arm_gripper_rclaw_joint
